File: Hardware/Tropic/sensor.kicad_sch (KiCad schematic)
At the start: 1 part, among them J2 68610414422

Commit message: Latest changes
Other:
- title: (none) -> Sensor
- moved on the sheet: J2
Changed lines of the file:
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@@
   (paper "A4")
   (title_block
+    (title "Sensor")
     (rev "1.0")
   )
-  (hierarchical_label "SCL" (shape input) (at 114.935 43.18 180) (fields_autoplaced)
+  (hierarchical_label "SCL" (shape input) (at 146.685 72.39 180) (fields_autoplaced)
     (effects (font (size 1.27 1.27)) (justify right))
   )
-  (hierarchical_label "SDA" (shape bidirectional) (at 114.935 40.64 180) (fields_autoplaced)
+  (hierarchical_label "SDA" (shape bidirectional) (at 146.685 69.85 180) (fields_autoplaced)
     (effects (font (size 1.27 1.27)) (justify right))
   )
-  (symbol (lib_id "power:+3.3V") (at 114.935 38.1 0) (unit 1)
+  (symbol (lib_id "power:+3.3V") (at 146.685 67.31 0) (unit 1)
     (in_bom yes) (on_board yes) (dnp no) (fields_autoplaced)
-    (property "Reference" "#PWR012" (at 114.935 41.91 0)
+    (property "Reference" "#PWR012" (at 146.685 71.12 0)
       (effects (font (size 1.27 1.27)) hide)
     )
-    (property "Value" "+3.3V" (at 114.935 34.155 0)
+    (property "Value" "+3.3V" (at 146.685 63.365 0)
       (effects (font (size 1.27 1.27)))
     )
-    (property "Footprint" "" (at 114.935 38.1 0)
+    (property "Footprint" "" (at 146.685 67.31 0)
       (effects (font (size 1.27 1.27)) hide)
     )
-    (property "Datasheet" "" (at 114.935 38.1 0)
+    (property "Datasheet" "" (at 146.685 67.31 0)
       (effects (font (size 1.27 1.27)) hide)
     )
@@
     )
   )
-  (symbol (lib_id "manul_tech:68610414422") (at 120.015 40.64 0) (mirror x) (unit 1)
+  (symbol (lib_id "manul_tech:68610414422") (at 151.765 69.85 0) (mirror x) (unit 1)
     (in_bom yes) (on_board yes) (dnp no)
-    (property "Reference" "J2" (at 119.126 42.934 0)
+    (property "Reference" "J2" (at 150.876 72.144 0)
       (effects (font (size 1.27 1.27)) (justify left))
     )
-    (property "Value" "68610414422" (at 119.126 40.886 0)
+    (property "Value" "68610414422" (at 150.876 70.096 0)
       (effects (font (size 1.27 1.27)) (justify left))
     )
-    (property "Footprint" "manul_tech:68610414422" (at 120.015 40.64 0)
+    (property "Footprint" "manul_tech:68610414422" (at 151.765 69.85 0)
       (effects (font (size 1.27 1.27)) (justify bottom) hide)
     )
-    (property "Datasheet" "" (at 120.015 40.64 0)
+    (property "Datasheet" "" (at 151.765 69.85 0)
       (effects (font (size 1.27 1.27)) hide)
     )
-    (property "internalRef" "" (at 120.015 40.64 0)
+    (property "internalRef" "" (at 151.765 69.85 0)
       (effects (font (size 1.27 1.27)) hide)
     )
-    (property "Manufacturer" "Wuerth Elektronik" (at 120.015 40.64 0)
+    (property "Manufacturer" "Wuerth Elektronik" (at 151.765 69.85 0)
       (effects (font (size 1.27 1.27)) hide)
     )
-    (property "MPN" "68610414422" (at 120.015 40.64 0)
+    (property "MPN" "68610414422" (at 151.765 69.85 0)
       (effects (font (size 1.27 1.27)) hide)
     )
@@
     )
   )
-  (symbol (lib_id "power:GND") (at 114.935 45.72 0) (unit 1)
+  (symbol (lib_id "power:GND") (at 146.685 74.93 0) (unit 1)
     (in_bom yes) (on_board yes) (dnp no) (fields_autoplaced)
-    (property "Reference" "#PWR013" (at 114.935 52.07 0)
+    (property "Reference" "#PWR013" (at 146.685 81.28 0)
       (effects (font (size 1.27 1.27)) hide)
     )
-    (property "Value" "GND" (at 114.935 49.665 0)
+    (property "Value" "GND" (at 146.685 78.875 0)
       (effects (font (size 1.27 1.27)))
     )
-    (property "Footprint" "" (at 114.935 45.72 0)
+    (property "Footprint" "" (at 146.685 74.93 0)
       (effects (font (size 1.27 1.27)) hide)
     )
-    (property "Datasheet" "" (at 114.935 45.72 0)
+    (property "Datasheet" "" (at 146.685 74.93 0)
       (effects (font (size 1.27 1.27)) hide)
     )
