File: Hardware/Tropic/Tropic.kicad_pcb (KiCad board)
At the start: 4 copper layers, 35.8 x 24.7 mm, 30 parts, among them J1 0734120114, J2 68610414422, J4 53309-1070, Q3 FDN340P, SW1 B3U-3000P, U1 ESP32-PICO-D4, U4 NCP1117ST33T3G

Commit message: Rework on components
Parts:
- removed C11, C12: 10uF, Capacitor_SMD:C_0402_1005Metric
- removed D1: PWR, LED_SMD:LED_0402_1005Metric
- removed D2: EXT_PWR, LED_SMD:LED_0402_1005Metric
- removed D3: 1N5819W, Diode_SMD:D_SOD-123
- removed D4: BATT_PWR, LED_SMD:LED_0402_1005Metric
- removed J4: 53309-1070, manul_tech:CON_533091070
- removed Q3: FDN340P, Package_TO_SOT_SMD:SOT-23
- removed U4: NCP1117ST33T3G, Package_TO_SOT_SMD:SOT-223-3_TabPin2
- added C6: 10uF, Capacitor_SMD:C_0603_1608Metric, F.Cu at (180.4, 39.4)
- added C7: 4.7uF, Capacitor_SMD:C_0603_1608Metric, F.Cu at (185.4, 39.1)
- added C8: 10uF, Capacitor_SMD:C_0402_1005Metric, F.Cu at (208.8, 18.4)
- added C9: 1uF, Capacitor_SMD:C_0402_1005Metric, F.Cu at (210.3, 17.2)
- added R10: 110K, Resistor_SMD:R_0402_1005Metric, F.Cu at (189.1, 39.9)
- added R11: 2K, Resistor_SMD:R_0402_1005Metric, F.Cu at (191.4, 31.9)
- added R13: TBD, Resistor_SMD:R_0402_1005Metric, F.Cu at (191.4, 33.0)
- added R14: 220R, Resistor_SMD:R_0402_1005Metric, F.Cu at (210.3, 16.2)
- added R15: 5.1K, Resistor_SMD:R_0402_1005Metric, F.Cu at (185.6, 25.0)
- added R16: 220R, Resistor_SMD:R_0402_1005Metric, F.Cu at (210.8, 24.5)
- added R17: 5.1K, Resistor_SMD:R_0402_1005Metric, F.Cu at (182.5, 25.0)
- added R18: 10K, Resistor_SMD:R_0402_1005Metric, F.Cu at (199.8, 18.3)
- added R9: 330K, Resistor_SMD:R_0402_1005Metric, F.Cu at (190.1, 41.0)
- added SW2: B3U-3000P, manul_tech:SW_B3U-3000P, F.Cu at (212.9, 25.7)
- added U2: ESP32-C3-WROOM-02U-N4, manul_tech:XCVR_ESP32-C3-WROOM-02U-N4, F.Cu at (202.5, 28.7)
- added U3: LM3671MF-3.3, Package_TO_SOT_SMD:SOT-23-5, F.Cu at (182.9, 39.5)
- C2: value TBD -> 100nF
- C3: value TBD -> 4.7uF; footprint Capacitor_SMD:C_0402_1005Metric -> Capacitor_SMD:C_0603_1608Metric
- C4: value 100nF -> 4.7uF; footprint Capacitor_SMD:C_0402_1005Metric -> Capacitor_SMD:C_0603_1608Metric
- C5: footprint Capacitor_SMD:C_0402_1005Metric -> Capacitor_SMD:C_0603_1608Metric
- J1: value 0734120114 -> 629722000214; footprint manul_tech:0734120114 -> manul_tech:629722000214
- L1: value TBD -> 2.2uH; footprint Inductor_SMD:L_0402_1005Metric -> manul_tech:CDRH2D14NP-2R2NC
- R12: value 100K -> 10K
- R6, R7: value 220R -> 27R
- R8: value 220R -> 10K
- SW1: moved to F.Cu
- U1: value ESP32-PICO-D4 -> MCP73871T-2CCI_ML; footprint Package_DFN_QFN:QFN-48-1EP_7x7mm_P0.5mm_EP5.3x5.3mm -> manul_tech:QFN50P400X400X100-21N
- moved L1 34.4 mm to (182.8, 43.8), turned to -90 degrees
- moved SW1 31.3 mm to (212.9, 17.9), turned to 90 degrees
- moved R8 30.5 mm to (204.8, 39.1)
- moved J1 26.5 mm to (184.0, 17.9), turned to 180 degrees
- moved C4 26.2 mm to (187.1, 39.1), turned to -90 degrees
- moved C5 25.2 mm to (186.7, 35.4), turned to 90 degrees
- moved C3 23.9 mm to (188.5, 32.7), turned to 180 degrees
- moved R12 21.4 mm to (208.3, 16.7)
- moved U1 19.3 mm to (190.1, 36.2), turned to 90 degrees
- moved R2 12.6 mm to (195.3, 40.5), turned to 0 degrees
- moved J2 12.3 mm to (196.3, 45.0)
- moved R3 7.66 mm to (197.3, 40.5), turned to 180 degrees
- moved R5 7.02 mm to (195.6, 17.8), turned to 0 degrees
- moved R1 6.72 mm to (206.8, 17.1), turned to 180 degrees
- moved C1 6.06 mm to (206.3, 18.4), turned to 180 degrees
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Connections:
- BATT1 pad 3: unconnected-(BATT1-NTC-Pad3) -> /Power Supply/NTC
- C2 pad 1: Net-(C2-Pad1) -> +3.3V
- C3 pad 1: Net-(U1-LNA_IN) -> +BATT
- C4 pad 1: +3.3V -> VDC
- C5 pad 1: +3.3V -> VBUS
- L1 pad 1: Net-(U1-LNA_IN) -> Net-(U3-SW)
- L1 pad 2: Net-(C2-Pad1) -> +3.3V
- R12 pad 1: VDC -> +3.3V
- R12 pad 2: GND -> /MCU/~{BOOT}
- R4 pad 2: /MCU/GPI35 -> /MCU/IO0
- R5 pad 1: /MCU/GPI35 -> /MCU/IO0
- R6 pad 1: +3.3V -> Net-(U2-IO18)
- R6 pad 2: Net-(D1-A) -> /MCU/USB_D-
- R7 pad 1: VDC -> Net-(U2-IO19)
- R7 pad 2: Net-(D2-A) -> /MCU/USB_D+
- R8 pad 1: Net-(R8-Pad1) -> +3.3V
- SW1 pad 1: Net-(R8-Pad1) -> GND
- SW1 pad 2: +BATT -> Net-(R14-Pad1)
- U1 pad 1: +3.3V -> VDC
- U1 pad 10: /MCU/GPI34 -> GND
- U1 pad 11: /MCU/GPI35 -> GND
- U1 pad 12: /MCU/GPIO32 -> Net-(U1-PROG3)
- U1 pad 13: /MCU/GPIO33 -> Net-(U1-PROG1)
- U1 pad 14: /MCU/GPIO25 -> +BATT
- U1 pad 15: /MCU/GPIO26 -> +BATT
- U1 pad 16: /MCU/GPIO27 -> +BATT
- U1 pad 17: /MCU/GPIO14 -> VBUS
- U1 pad 18: /MCU/GPIO12 -> VBUS
- U1 pad 19: +3.3V -> VBUS
- U1 pad 2: Net-(U1-LNA_IN) -> Net-(U1-VPCC)
- U1 pad 20: /MCU/GPIO13 -> VDC
- U1 pad 21: /MCU/GPIO15 -> GND
- U1 pad 3: +3.3V -> GND
- U1 pad 4: +3.3V -> VBUS
- U1 pad 5: unconnected-(U1-SENSOR_VP-Pad5) -> /Power Supply/NTC
- U1 pad 6: unconnected-(U1-SENSOR_CAPP-Pad6) -> /MCU/IO3
- U1 pad 7: unconnected-(U1-SENSOR_CAPN-Pad7) -> /MCU/IO4
- U1 pad 8: unconnected-(U1-SENSOR_VN-Pad8) -> /MCU/IO1
- U1 pad 9: /MCU/EN -> VBUS
Routing:
- net /MCU/TX: track 33.4 -> 0.00 mm, vias 2 -> 0
- net /MCU/RX: track 33.2 -> 0.00 mm, vias 2 -> 0
- net /MCU/GPI35: track 28.7 -> 0.00 mm, vias 1 -> 0
- net /MCU/EN: track 26.9 -> 0.00 mm, vias 2 -> 0
- net /MCU/IO0: track 23.3 -> 0.00 mm, vias 2 -> 0
- net /Power Supply/NTC: track 0.00 -> 22.5 mm, vias 0 -> 1
- net /MCU/SCL: track 24.4 -> 3.20 mm, vias 0 -> 1
- net +3.3V: track 25.4 -> 5.11 mm, vias 14 -> 7
- net /MCU/SDA: track 23.5 -> 3.44 mm, vias 2 -> 1
- net /MCU/~{BOOT}: track 0.00 -> 15.9 mm
- net +BATT: track 15.5 -> 0.00 mm, vias 1 -> 0
- net Net-(D3-K): track 13.0 -> 0.00 mm
- net VBUS: track 0.00 -> 8.98 mm, vias 0 -> 4
- net VDC: track 10.5 -> 1.53 mm, vias 0 -> 1
- net Net-(R8-Pad1): track 4.10 -> 0.00 mm, vias 1 -> 0
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- added copper zone on F.Cu, net +BATT
- added copper zone on F.Cu, net VBUS
- removed copper zone on In1.Cu, net +3.3V
- removed copper zone on B.Cu, net GND
- removed copper zone on F.Cu, net GND
- removed copper zone on In2.Cu, net GND
Other:
- board size 35.8 x 24.7 mm -> 35.8 x 31.6 mm
- board text removed: "3V3"
- board text removed: "BAT"
- board text removed: "EXT"
