File: Hardware/Tropic/Tropic.kicad_sch (KiCad schematic)
At the start: 0 parts

Commit message: Latest changes
Other:
- removed sheet GPIO
Changed lines of the file:
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@@
-    )
-  )
-  (sheet (at 160.02 54.61) (size 12.7 33.02) (fields_autoplaced)
-    (stroke (width 0.1524) (type solid))
-    (fill (color 0 0 0 0.0000))
-    (property "Sheetname" "GPIO" (at 160.02 53.8984 0)
-      (effects (font (size 1.27 1.27)) (justify left bottom))
-    )
-    (property "Sheetfile" "gpio.kicad_sch" (at 160.02 88.2146 0)
-      (effects (font (size 1.27 1.27)) (justify left top))
-    )
-    (instances
-      (project "Tropic"
-        (path "/03cbb5e4-b4a9-4ace-b6fb-ea1f35182954" (page "6"))
-      )
     )
   )

Commit message: Rework on components
Other:
- sheet MCU ports: added IO1, IO3, IO4, USB_D+, USB_D-; removed EN, GPI34, GPI35, GPIO10, GPIO12, GPIO13, GPIO14, GPIO15, GPIO18, GPIO19, GPIO23, GPIO25, GPIO26, GPIO27, GPIO32, GPIO33, GPIO4, GPIO5, GPIO9, RX, TX
- sheet Power Supply ports: added STAT2, ~{LBO}, ~{PG}; removed none
- sheet Program Interface ports: added USB_D+, USB_D-; removed EN, IO0, RX, TX
Changed lines of the file:
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@@
     (rev "1.0")
   )
-  (wire (pts (xy 109.22 51.435) (xy 121.92 51.435))
+  (wire (pts (xy 109.22 56.515) (xy 121.92 56.515))
+    (stroke (width 0) (type default))
+  )
+  (wire (pts (xy 109.22 45.085) (xy 121.92 45.085))
+    (stroke (width 0) (type default))
+  )
+  (wire (pts (xy 109.22 46.99) (xy 121.92 46.99))
+    (stroke (width 0) (type default))
+  )
+  (wire (pts (xy 147.955 47.625) (xy 160.02 47.625))
+    (stroke (width 0) (type default))
+  )
+  (wire (pts (xy 109.22 64.135) (xy 121.92 64.135))
     (stroke (width 0) (type default))
   )
@@
     (stroke (width 0) (type default))
   )
-  (wire (pts (xy 109.22 45.72) (xy 121.92 45.72))
-    (stroke (width 0) (type default))
-  )
-  (wire (pts (xy 147.955 47.625) (xy 160.02 47.625))
-    (stroke (width 0) (type default))
-  )
-  (wire (pts (xy 109.22 49.53) (xy 121.92 49.53))
+  (wire (pts (xy 109.22 59.055) (xy 121.92 59.055))
     (stroke (width 0) (type default))
   )
@@
     (stroke (width 0) (type default))
   )
-  (wire (pts (xy 109.22 47.625) (xy 121.92 47.625))
-    (stroke (width 0) (type default))
-  )
-  (sheet (at 121.92 43.18) (size 26.035 44.45) (fields_autoplaced)
+  (sheet (at 121.92 43.18) (size 26.035 26.035) (fields_autoplaced)
     (stroke (width 0.1524) (type solid))
     (fill (color 0 0 0 0.0000))
@@
       (effects (font (size 1.27 1.27)) (justify left bottom))
     )
-    (property "Sheetfile" "mcu.kicad_sch" (at 121.92 88.2146 0)
+    (property "Sheetfile" "mcu.kicad_sch" (at 121.92 69.7996 0)
       (effects (font (size 1.27 1.27)) (justify left top))
-    )
-    (pin "EN" input (at 121.92 45.72 180)
-      (effects (font (size 1.27 1.27)) (justify left))
-    )
-    (pin "IO0" input (at 121.92 47.625 180)
-      (effects (font (size 1.27 1.27)) (justify left))
-    )
-    (pin "TX" output (at 121.92 49.53 180)
-      (effects (font (size 1.27 1.27)) (justify left))
-    )
-    (pin "RX" input (at 121.92 51.435 180)
-      (effects (font (size 1.27 1.27)) (justify left))
     )
     (pin "SCL" output (at 147.955 45.72 0)
@@
       (effects (font (size 1.27 1.27)) (justify right))
     )
-    (pin "GPIO19" bidirectional (at 147.955 69.215 0)
-      (effects (font (size 1.27 1.27)) (justify right))
-    )
-    (pin "GPIO18" bidirectional (at 147.955 71.12 0)
-      (effects (font (size 1.27 1.27)) (justify right))
-    )
-    (pin "GPIO15" bidirectional (at 147.955 73.025 0)
-      (effects (font (size 1.27 1.27)) (justify right))
-    )
-    (pin "GPIO14" bidirectional (at 147.955 74.93 0)
-      (effects (font (size 1.27 1.27)) (justify right))
-    )
-    (pin "GPIO13" bidirectional (at 147.955 76.835 0)
-      (effects (font (size 1.27 1.27)) (justify right))
-    )
-    (pin "GPIO12" bidirectional (at 147.955 78.74 0)
-      (effects (font (size 1.27 1.27)) (justify right))
-    )
-    (pin "GPIO10" bidirectional (at 147.955 80.645 0)
-      (effects (font (size 1.27 1.27)) (justify right))
-    )
-    (pin "GPIO9" bidirectional (at 147.955 82.55 0)
-      (effects (font (size 1.27 1.27)) (justify right))
-    )
-    (pin "GPIO5" bidirectional (at 147.955 84.455 0)
-      (effects (font (size 1.27 1.27)) (justify right))
-    )
-    (pin "GPIO4" bidirectional (at 147.955 86.36 0)
-      (effects (font (size 1.27 1.27)) (justify right))
-    )
-    (pin "GPIO25" bidirectional (at 147.955 65.405 0)
-      (effects (font (size 1.27 1.27)) (justify right))
-    )
-    (pin "GPIO23" bidirectional (at 147.955 67.31 0)
-      (effects (font (size 1.27 1.27)) (justify right))
-    )
-    (pin "GPIO27" bidirectional (at 147.955 61.595 0)
-      (effects (font (size 1.27 1.27)) (justify right))
-    )
-    (pin "GPIO32" bidirectional (at 147.955 59.69 0)
-      (effects (font (size 1.27 1.27)) (justify right))
-    )
-    (pin "GPIO33" bidirectional (at 147.955 57.785 0)
-      (effects (font (size 1.27 1.27)) (justify right))
-    )
-    (pin "GPI35" bidirectional (at 121.92 61.595 180)
+    (pin "USB_D-" bidirectional (at 121.92 45.085 180)
       (effects (font (size 1.27 1.27)) (justify left))
     )
-    (pin "GPI34" bidirectional (at 147.955 55.88 0)
-      (effects (font (size 1.27 1.27)) (justify right))
+    (pin "USB_D+" bidirectional (at 121.92 46.99 180)
+      (effects (font (size 1.27 1.27)) (justify left))
     )
-    (pin "GPIO26" bidirectional (at 147.955 63.5 0)
-      (effects (font (size 1.27 1.27)) (justify right))
+    (pin "IO0" input (at 121.92 56.515 180)
+      (effects (font (size 1.27 1.27)) (justify left))
+    )
+    (pin "IO1" input (at 121.92 59.055 180)
+      (effects (font (size 1.27 1.27)) (justify left))
+    )
+    (pin "IO3" input (at 121.92 61.595 180)
+      (effects (font (size 1.27 1.27)) (justify left))
+    )
+    (pin "IO4" input (at 121.92 64.135 180)
+      (effects (font (size 1.27 1.27)) (justify left))
     )
     (instances
@@
     )
   )
-  (sheet (at 96.52 59.69) (size 12.7 3.81) (fields_autoplaced)
+  (sheet (at 96.52 54.61) (size 12.7 14.605) (fields_autoplaced)
     (stroke (width 0.1524) (type solid))
     (fill (color 0 0 0 0.0000))
-    (property "Sheetname" "Power Supply" (at 96.52 58.9784 0)
+    (property "Sheetname" "Power Supply" (at 96.52 53.8984 0)
       (effects (font (size 1.27 1.27)) (justify left bottom))
     )
-    (property "Sheetfile" "psu.kicad_sch" (at 96.52 64.0846 0)
+    (property "Sheetfile" "psu.kicad_sch" (at 96.52 69.7996 0)
       (effects (font (size 1.27 1.27)) (justify left top))
     )
-    (pin "BATT" output (at 109.22 61.595 0)
+    (pin "BATT" output (at 109.22 56.515 0)
+      (effects (font (size 1.27 1.27)) (justify right))
+    )
+    (pin "~{LBO}" output (at 109.22 59.055 0)
+      (effects (font (size 1.27 1.27)) (justify right))
+    )
+    (pin "~{PG}" output (at 109.22 61.595 0)
+      (effects (font (size 1.27 1.27)) (justify right))
+    )
+    (pin "STAT2" output (at 109.22 64.135 0)
       (effects (font (size 1.27 1.27)) (justify right))
     )
@@
     )
   )
-  (sheet (at 96.52 43.18) (size 12.7 10.16) (fields_autoplaced)
+  (sheet (at 96.52 43.18) (size 12.7 5.715) (fields_autoplaced)
     (stroke (width 0.1524) (type solid))
     (fill (color 0 0 0 0.0000))
@@
       (effects (font (size 1.27 1.27)) (justify left bottom))
     )
-    (property "Sheetfile" "flash.kicad_sch" (at 96.52 53.9246 0)
+    (property "Sheetfile" "flash.kicad_sch" (at 96.52 49.4796 0)
       (effects (font (size 1.27 1.27)) (justify left top))
     )
-    (pin "TX" input (at 109.22 49.53 0)
+    (pin "USB_D+" bidirectional (at 109.22 46.99 0)
       (effects (font (size 1.27 1.27)) (justify right))
     )
-    (pin "RX" output (at 109.22 51.435 0)
+    (pin "USB_D-" bidirectional (at 109.22 45.085 0)
       (effects (font (size 1.27 1.27)) (justify right))
     )
-    (pin "EN" output (at 109.22 45.72 0)
-      (effects (font (size 1.27 1.27)) (justify right))
-    )
-    (pin "IO0" output (at 109.22 47.625 0)
-      (effects (font (size 1.27 1.27)) (justify right))
-    )
