File: Hardware/Tropic/mcu.kicad_sch (KiCad schematic)
At the start: 16 parts, among them J1 0734120114, U1 ESP32-PICO-D4

Commit message: Removed doubled Pi Matching and add LED for voltage monitoring
Parts:
- removed C13, C14: TBD, Capacitor_SMD:C_0402_1005Metric, symbol Device:C_Small
- removed E1: 2450AT42E010BE, manul_tech:XDCR_2450AT42E010BE, symbol manul_tech:2450AT42E010BE
- removed JP1: Antenna Selector, Jumper:SolderJumper-3_P1.3mm_Open_RoundedPad1.0x1.5mm, symbol Jumper:Jumper_3_Bridged12
- removed L2: TBD, Inductor_SMD:L_0402_1005Metric, symbol Device:L_Small
Connections:
- net at C2.1, L1.2: now also J1.1
Other:
- moved on the sheet: J1, L1

Commit message: Completed design V1
Other:
- moved on the sheet: C2, C3
Changed lines of the file:
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@@
     (rev "1.0")
   )
-  (junction (at 223.52 45.72) (diameter 0) (color 0 0 0 0)
-  )
   (junction (at 112.395 45.72) (diameter 0) (color 0 0 0 0)
   )
@@
   (junction (at 144.78 40.64) (diameter 0) (color 0 0 0 0)
   )
+  (junction (at 205.74 45.72) (diameter 0) (color 0 0 0 0)
+  )
+  (junction (at 215.9 45.72) (diameter 0) (color 0 0 0 0)
+  )
   (junction (at 146.05 40.64) (diameter 0) (color 0 0 0 0)
   )
   (junction (at 147.32 40.64) (diameter 0) (color 0 0 0 0)
-  )
-  (junction (at 198.755 45.72) (diameter 0) (color 0 0 0 0)
   )
   (junction (at 130.175 35.56) (diameter 0) (color 0 0 0 0)
@@
     (stroke (width 0) (type default))
   )
-  (wire (pts (xy 213.36 45.72) (xy 223.52 45.72))
+  (wire (pts (xy 213.36 45.72) (xy 215.9 45.72))
     (stroke (width 0) (type default))
   )
@@
     (stroke (width 0) (type default))
   )
+  (wire (pts (xy 205.74 45.72) (xy 208.28 45.72))
+    (stroke (width 0) (type default))
+  )
   (wire (pts (xy 147.32 121.92) (xy 147.32 123.19))
     (stroke (width 0) (type default))
@@
     (stroke (width 0) (type default))
   )
-  (wire (pts (xy 167.64 45.72) (xy 198.755 45.72))
+  (wire (pts (xy 167.64 45.72) (xy 205.74 45.72))
     (stroke (width 0) (type default))
   )
@@
     (stroke (width 0) (type default))
   )
-  (wire (pts (xy 223.52 45.72) (xy 231.775 45.72))
+  (wire (pts (xy 215.9 45.72) (xy 231.775 45.72))
     (stroke (width 0) (type default))
   )
@@
   )
   (wire (pts (xy 167.64 58.42) (xy 183.515 58.42))
-    (stroke (width 0) (type default))
-  )
-  (wire (pts (xy 198.755 45.72) (xy 208.28 45.72))
     (stroke (width 0) (type default))
   )
@@
     )
   )
-  (symbol (lib_id "Device:C_Small") (at 198.755 48.26 0) (mirror y) (unit 1)
+  (symbol (lib_id "Device:C_Small") (at 205.74 48.26 0) (mirror y) (unit 1)
     (in_bom yes) (on_board yes) (dnp no)
-    (property "Reference" "C3" (at 196.4309 47.2423 0)
-      (effects (font (size 1.27 1.27)) (justify left))
-    )
-    (property "Value" "TBD" (at 196.4309 49.2903 0)
-      (effects (font (size 1.27 1.27)) (justify left))
-    )
-    (property "Footprint" "Capacitor_SMD:C_0402_1005Metric" (at 198.755 48.26 0)
-      (effects (font (size 1.27 1.27)) hide)
-    )
-    (property "Datasheet" "~" (at 198.755 48.26 0)
+    (property "Reference" "C3" (at 203.4159 47.2423 0)
+      (effects (font (size 1.27 1.27)) (justify left))
+    )
+    (property "Value" "TBD" (at 203.4159 49.2903 0)
+      (effects (font (size 1.27 1.27)) (justify left))
+    )
+    (property "Footprint" "Capacitor_SMD:C_0402_1005Metric" (at 205.74 48.26 0)
+      (effects (font (size 1.27 1.27)) hide)
+    )
+    (property "Datasheet" "~" (at 205.74 48.26 0)
       (effects (font (size 1.27 1.27)) hide)
     )
@@
     )
   )
-  (symbol (lib_id "power:GND") (at 198.755 50.8 0) (unit 1)
-    (in_bom yes) (on_board yes) (dnp no) (fields_autoplaced)
-    (property "Reference" "#PWR04" (at 198.755 57.15 0)
-      (effects (font (size 1.27 1.27)) hide)
-    )
-    (property "Value" "GND" (at 198.755 54.745 0)
-      (effects (font (size 1.27 1.27)))
-    )
-    (property "Footprint" "" (at 198.755 50.8 0)
-      (effects (font (size 1.27 1.27)) hide)
-    )
-    (property "Datasheet" "" (at 198.755 50.8 0)
+  (symbol (lib_id "power:GND") (at 205.74 50.8 0) (unit 1)
+    (in_bom yes) (on_board yes) (dnp no) (fields_autoplaced)
+    (property "Reference" "#PWR04" (at 205.74 57.15 0)
+      (effects (font (size 1.27 1.27)) hide)
+    )
+    (property "Value" "GND" (at 205.74 54.745 0)
+      (effects (font (size 1.27 1.27)))
+    )
+    (property "Footprint" "" (at 205.74 50.8 0)
+      (effects (font (size 1.27 1.27)) hide)
+    )
+    (property "Datasheet" "" (at 205.74 50.8 0)
       (effects (font (size 1.27 1.27)) hide)
     )
@@
     )
   )
-  (symbol (lib_id "Device:C_Small") (at 223.52 48.26 0) (unit 1)
-    (in_bom yes) (on_board yes) (dnp no) (fields_autoplaced)
-    (property "Reference" "C2" (at 225.8441 47.2423 0)
-      (effects (font (size 1.27 1.27)) (justify left))
-    )
-    (property "Value" "TBD" (at 225.8441 49.2903 0)
-      (effects (font (size 1.27 1.27)) (justify left))
-    )
-    (property "Footprint" "Capacitor_SMD:C_0402_1005Metric" (at 223.52 48.26 0)
-      (effects (font (size 1.27 1.27)) hide)
-    )
-    (property "Datasheet" "~" (at 223.52 48.26 0)
+  (symbol (lib_id "Device:C_Small") (at 215.9 48.26 0) (unit 1)
+    (in_bom yes) (on_board yes) (dnp no) (fields_autoplaced)
+    (property "Reference" "C2" (at 218.2241 47.2423 0)
+      (effects (font (size 1.27 1.27)) (justify left))
+    )
+    (property "Value" "TBD" (at 218.2241 49.2903 0)
+      (effects (font (size 1.27 1.27)) (justify left))
+    )
+    (property "Footprint" "Capacitor_SMD:C_0402_1005Metric" (at 215.9 48.26 0)
+      (effects (font (size 1.27 1.27)) hide)
+    )
+    (property "Datasheet" "~" (at 215.9 48.26 0)
       (effects (font (size 1.27 1.27)) hide)
     )
@@
     )
   )
-  (symbol (lib_id "power:GND") (at 223.52 50.8 0) (unit 1)
-    (in_bom yes) (on_board yes) (dnp no) (fields_autoplaced)
-    (property "Reference" "#PWR05" (at 223.52 57.15 0)
-      (effects (font (size 1.27 1.27)) hide)
-    )
-    (property "Value" "GND" (at 223.52 54.745 0)
-      (effects (font (size 1.27 1.27)))
-    )
-    (property "Footprint" "" (at 223.52 50.8 0)
-      (effects (font (size 1.27 1.27)) hide)
-    )
-    (property "Datasheet" "" (at 223.52 50.8 0)
-      (effects (font (size 1.27 1.27)) hide)
-    )
+  (symbol (lib_id "power:GND") (at 215.9 50.8 0) (unit 1)
+    (in_bom yes) (on_board yes) (dnp no) (fields_autoplaced)
+    (property "Reference" "#PWR05" (at 215.9 57.15 0)
+      (effects (font (size 1.27 1.27)) hide)
+    )
+    (property "Value" "GND" (at 215.9 54.745 0)
+      (effects (font (size 1.27 1.27)))
+    )
+    (property "Footprint" "" (at 215.9 50.8 0)
+      (effects (font (size 1.27 1.27)) hide)
+    )
+    (property "Datasheet" "" (at 215.9 50.8 0)
+      (effects (font (size 1.27 1.27)) hide)
+    )

Commit message: Latest changes
Other:
- title: (none) -> ESP32 
Changed lines of the file:
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@@
   (paper "A4")
   (title_block
+    (title "ESP32 ")
     (rev "1.0")
   )

Commit message: Rework on components
Parts:
- removed C3: TBD, Capacitor_SMD:C_0402_1005Metric, symbol Device:C_Small
- removed C4: 100nF, Capacitor_SMD:C_0402_1005Metric, symbol Device:C_Small
- removed C5: 10uF, Capacitor_SMD:C_0402_1005Metric, symbol Device:C_Small
- removed J1: 0734120114, manul_tech:0734120114, symbol manul_tech:0734120114
- removed L1: TBD, Inductor_SMD:L_0402_1005Metric, symbol Device:L_Small
- removed U1: ESP32-PICO-D4, Package_DFN_QFN:QFN-48-1EP_7x7mm_P0.5mm_EP5.3x5.3mm, symbol RF_Module:ESP32-PICO-D4
- added C8: 10uF, Capacitor_SMD:C_0402_1005Metric, symbol Device:C_Small
- added C9: 1uF, Capacitor_SMD:C_0402_1005Metric, symbol Device:C_Small
- added R12, R18, R8: 10K, Resistor_SMD:R_0402_1005Metric, symbol Device:R_Small
- added R14, R16: 220R, Resistor_SMD:R_0402_1005Metric, symbol Device:R_Small
- added R6, R7: 27R, Resistor_SMD:R_0402_1005Metric, symbol Device:R_Small
- added SW1, SW2: B3U-3000P, manul_tech:SW_B3U-3000P, symbol manul_tech:B3U-3000P
- added U2: ESP32-C3-WROOM-02U-N4, manul_tech:XCVR_ESP32-C3-WROOM-02U-N4, symbol manul_tech:ESP32-C3-WROOM-02U-N4
- C2: value TBD -> 100nF; internalRef (none) -> 1.03.013
Connections:
- net +3.3V: now also C2.1, C8.1, R12.1, R18.1, R8.1, U2.1 (3V3)
- net EN: now also R16.2, U2.2 (EN)
- net GND: now also C8.2, C9.2, SW1.1, SW2.1, U2.19_1 (GND), U2.19_2 (GND), U2.19_3 (GND), U2.19_4 (GND), U2.19_5 (GND), U2.19_6 (GND), U2.19_7 (GND), U2.19_8 (GND), U2.19_9 (GND), U2.9 (GND)
- net IO0: now also U2.18 (IO0)
- net SCL: now also U2.5 (IO6)
- net SDA: now also U2.4 (IO5)
- new net: R16.1, SW2.2
- new net: R6.1, U2.13 (IO18)
- new net: R7.1, U2.14 (IO19)
- new net: R8.2, U2.16 (IO2)
- new net: R14.1, SW1.2
- new net IO1: U2.17 (IO1)
- new net IO3: U2.15 (IO3)
- new net IO4: U2.3 (IO4)
- new net IO8: R18.2, U2.7 (IO8)
- new net USB_D+: R7.2
- new net USB_D-: R6.2
- new net ~{BOOT}: C9.1, R12.2, R14.2, U2.8 (IO9)
- no-connect marks 12 -> 4
Other:
- moved on the sheet: C1, R1, R2, R3
