File: Hardware/Tropic/psu.kicad_sch (KiCad schematic)
At the start: 16 parts, among them Q3 FDN340P, SW1 B3U-3000P, U4 NCP1117ST33T3G

Commit message: Completed design V1
Parts:
- added D5: 1N5819W, Diode_SMD:D_SOD-123, symbol manul_tech:1N5819W
Connections:
- net +BATT: now also D5.1 (K); no longer BATT1.1 (B+)
- new net: BATT1.1 (B+), D5.2 (A)
Changed lines of the file:
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@@
     )
   )
-  (symbol (lib_id "power:+BATT") (at 192.405 57.15 0) (mirror y) (unit 1)
-    (in_bom yes) (on_board yes) (dnp no) (fields_autoplaced)
-    (property "Reference" "#PWR044" (at 192.405 60.96 0)
-      (effects (font (size 1.27 1.27)) hide)
-    )
-    (property "Value" "+BATT" (at 192.405 53.205 0)
-      (effects (font (size 1.27 1.27)))
-    )
-    (property "Footprint" "" (at 192.405 57.15 0)
-      (effects (font (size 1.27 1.27)) hide)
-    )
-    (property "Datasheet" "" (at 192.405 57.15 0)
+  (symbol (lib_id "power:+BATT") (at 200.025 57.15 0) (mirror y) (unit 1)
+    (in_bom yes) (on_board yes) (dnp no) (fields_autoplaced)
+    (property "Reference" "#PWR044" (at 200.025 60.96 0)
+      (effects (font (size 1.27 1.27)) hide)
+    )
+    (property "Value" "+BATT" (at 200.025 53.205 0)
+      (effects (font (size 1.27 1.27)))
+    )
+    (property "Footprint" "" (at 200.025 57.15 0)
+      (effects (font (size 1.27 1.27)) hide)
+    )
+    (property "Datasheet" "" (at 200.025 57.15 0)
       (effects (font (size 1.27 1.27)) hide)
     )
@@
         )
       )
+    )
+  )
+  (symbol (lib_id "manul_tech:1N5819W") (at 196.215 57.15 0) (mirror y) (unit 1)
+    (in_bom yes) (on_board yes) (dnp no)
+    (property "Reference" "D5" (at 196.215 66.04 0)
+      (effects (font (size 1.27 1.27)))
+    )
+    (property "Value" "1N5819W" (at 198.755 63.5 0)
+      (effects (font (size 1.27 1.27)))
+    )
+    (property "Footprint" "Diode_SMD:D_SOD-123" (at 196.215 62.23 0)
+      (effects (font (size 1.27 1.27)) hide)
+    )
+    (property "Datasheet" "~" (at 196.215 62.23 0)
+      (effects (font (size 1.27 1.27)) hide)
+    )
+    (property "internalRef" "4.02.001" (at 198.755 60.96 0)
+      (effects (font (size 1.27 1.27)))
+    )
+    (property "MPN" "1N5819HW-7-F" (at 196.215 57.15 0)
+      (effects (font (size 1.27 1.27)) hide)
+    )
+    (pin "1")
+    (pin "2")
+    (instances
+      (project "Tropic"
+        (path "/03cbb5e4-b4a9-4ace-b6fb-ea1f35182954/b474f81d-bdf0-4c8f-a328-174e1d69093f"
+          (reference "D5") (unit 1)
+        )
+      )
+      (project "ESP_Temp_Watchdog"
+        (path "/deef4040-926c-4ef4-8894-27bba8836b5a/00000000-0000-0000-0000-0000615f0d56"
+          (reference "D1") (unit 1)
+        )
+      )

Commit message: Latest changes
Other:
- title: Power Supply -> Power Supply and status LED
Changed lines of the file:
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@@
   (paper "A4")
   (title_block
-    (title "Power Supply")
+    (title "Power Supply and status LED")
     (rev "1.0")
   )

Commit message: Rework on components
Parts:
- removed C11, C12: 10uF, Capacitor_SMD:C_0402_1005Metric, symbol Device:C_Small
- removed D1: PWR, LED_SMD:LED_0402_1005Metric, symbol Device:LED_Small
- removed D2: EXT_PWR, LED_SMD:LED_0402_1005Metric, symbol Device:LED_Small
- removed D3: 1N5819W, Diode_SMD:D_SOD-123, symbol manul_tech:1N5819W
- removed D4: BATT_PWR, LED_SMD:LED_0402_1005Metric, symbol Device:LED_Small
- removed Q3: FDN340P, Package_TO_SOT_SMD:SOT-23, symbol manul_tech:FDN340P
- removed R12: 100K, Resistor_SMD:R_0402_1005Metric, symbol Device:R_Small
- removed R6, R7, R8: 220R, Resistor_SMD:R_0402_1005Metric, symbol Device:R_Small
- removed SW1: B3U-3000P, SW_B3U-3000P, symbol manul_tech:B3U-3000P
- removed U4: NCP1117ST33T3G, Package_TO_SOT_SMD:SOT-223-3_TabPin2, symbol manul_tech:NCP1117ST33T3G
- added C3, C4, C7: 4.7uF, Capacitor_SMD:C_0603_1608Metric, symbol Device:C_Small
- added C5, C6: 10uF, Capacitor_SMD:C_0603_1608Metric, symbol Device:C_Small
- added L1: 2.2uH, manul_tech:CDRH2D14NP-2R2NC, symbol Device:L_Small
- added R10: 110K, Resistor_SMD:R_0402_1005Metric, symbol Device:R_Small
- added R11: 2K, Resistor_SMD:R_0402_1005Metric, symbol Device:R_Small
- added R13: TBD, Resistor_SMD:R_0402_1005Metric, symbol Device:R_Small
- added R9: 330K, Resistor_SMD:R_0402_1005Metric, symbol Device:R_Small
- added U1: MCP73871T-2CCI_ML, manul_tech:QFN50P400X400X100-21N, symbol manul_tech:MCP73871T-2CCI_ML
- added U3: LM3671MF-3.3, Package_TO_SOT_SMD:SOT-23-5, symbol manul_tech:LM3671MF-3.3
Connections:
- net +3.3V: now also C6.1, L1.2, U3.4 (FB)
- net +BATT: now also C3.1, U1.14 (VBAT), U1.15 (VBAT), U1.16 (VBAT_SENSE)
- net GND: now also C3.2, C4.2, C5.2, C6.2, C7.2, R10.2, R11.2, R13.2, U1.10 (VSS), U1.11 (VSS), U1.21 (EP), U1.3 (SEL), U3.2 (GND)
- net VDC: now also C4.1, C7.1, U1.1 (OUT), U1.20 (OUT), U3.1 (VIN), U3.3 (EN)
- net NTC: now reaches BATT1.3 (NTC)
- net NTC: now also U1.5 (THERM)
- new net: L1.1, U3.5 (SW)
- new net: R10.1, R9.2, U1.2 (VPCC)
- new net: R11.1, U1.13 (PROG1)
- new net: R13.1, U1.12 (PROG3)
- new net STAT2: U1.7 (STAT2)
- new net VBUS: C5.1, R9.1, U1.17 (CE), U1.18 (IN), U1.19 (IN), U1.4 (PROG2), U1.9 (~{TE})
- new net ~{LBO}: U1.8 (STAT1/~{LBO})
- new net ~{PG}: U1.6 (~{PG})
- no-connect marks 2 -> 1
Other:
- moved on the sheet: BATT1
