File: Hardware/Switch Board/mcu.kicad_sch (KiCad schematic)
At the start: 0 parts

Commit message: Completed Power Supply scheamatic + started to place components
Parts:
- added C2: 1uF, Capacitor_SMD:C_0402_1005Metric, symbol Device:C_Small
- added C3: 100nF, Capacitor_SMD:C_0402_1005Metric, symbol Device:C_Small
- added R1: 10K, Capacitor_SMD:C_0402_1005Metric, symbol Device:R_Small
- added U1: ESP32-WROOM-32UE_(16MB), manul_tech:XCVR_ESP32-WROOM-32UE_(16MB), symbol manul_tech:ESP32-WROOM-32UE_(16MB)
Connections:
- new net: U1.17 (NC), U1.18 (NC), U1.19 (NC), U1.20 (NC), U1.21 (NC), U1.22 (NC)
- new net +3V3: C3.1, R1.1, U1.2 (3V3)
- new net BOOT: U1.25 (IO0)
- new net EN: C2.1, R1.2, U1.3 (EN)
- new net GND: C2.2, C3.2, U1.1 (GND), U1.15 (GND), U1.38 (GND), U1.39_1 (GND), U1.39_2 (GND), U1.39_3 (GND), U1.39_4 (GND), U1.39_5 (GND), U1.39_6 (GND), U1.39_7 (GND), U1.39_8 (GND), U1.39_9 (GND)
- new net I34: U1.6 (IO34)
- new net I35: U1.7 (IO35)
- new net IO12: U1.14 (IO12)
- new net IO13: U1.16 (IO13)
- new net IO14: U1.13 (IO14)
- new net IO15: U1.23 (IO15)
- new net IO16: U1.27 (IO16)
- new net IO17_EMAC_CLK_OUT_180: U1.28 (IO17)
- new net IO18_MDIO: U1.30 (IO18)
- new net IO19_EMAC_TXD0: U1.31 (IO19)
- new net IO2: U1.24 (IO2)
- new net IO21_EMAC_TX_EN: U1.33 (IO21)
- new net IO22_EMAC_TXD1: U1.36 (IO22)
- new net IO23_MDC: U1.37 (IO23)
- new net IO25_EMAC_RXD0: U1.10 (IO25)
- new net IO26_EMAC_RXD1: U1.11 (IO26)
- new net IO27_EMAC_RX_CRS_DV: U1.12 (IO27)
- new net IO33: U1.9 (IO33)
- new net IO4: U1.26 (IO4)
- new net IO5_PHY_PWR: U1.29 (IO5)
- new net RLY_TGL: U1.8 (IO32)
- new net RX0: U1.34 (RXD0)
- new net TX0: U1.35 (TXD0)
- no-connect marks 0 -> 2
